File: pcb/main.brd (EAGLE design)
At the start: 62.2 x 49.2 mm, 19 parts, among them IC1 PCF8574P, U1 BMP280

Commit message: Update pcb files
Parts:
- removed DIS1: TUXGR_16X2_R2, display-lcd:TUXGR_16X2_R2
- moved R9 28.2 mm to (112.2, 25.2), turned to 270 degrees
- moved R2 24.6 mm to (117.4, 25.2), turned to 270 degrees
- moved R1 22.1 mm to (123.6, 24.2), turned to 270 degrees
- moved R6 20.9 mm to (130.7, 24.3), turned to 90 degrees
- moved U$1 14.1 mm to (104.0, 44.3), flipped to the bottom, turned to 90 degrees
- moved R10 14.0 mm to (91.4, 46.0)
- moved R11 14.0 mm to (91.4, 51.1)
- moved R5 14.0 mm to (91.4, 40.9)
- moved C1 14.0 mm to (97.4, 24.1)
- moved R7 13.8 mm to (131.0, 36.3), turned to 90 degrees
- moved JP2 13.6 mm to (109.5, 60.5)
- moved C2 12.2 mm to (103.4, 54.1)
- moved R4 11.7 mm to (106.7, 25.5), turned to 90 degrees
- moved R3 9.86 mm to (91.0, 35.4)
- moved U1 9.71 mm to (103.8, 34.7), flipped to the bottom, turned to 90 degrees
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Connections:
- net GND: no longer DIS1.1, DIS1.10, DIS1.16, DIS1.7, DIS1.8, DIS1.9
- net N$1: no longer DIS1.14
- net N$12: no longer DIS1.3
- net N$14: no longer DIS1.15
- net N$2: no longer DIS1.13
- net N$3: no longer DIS1.12
- net N$4: no longer DIS1.11
- net N$5: no longer DIS1.4
- net N$7: no longer DIS1.5
- net N$8: no longer DIS1.6
- net VCC: no longer DIS1.2
Routing:
- net GND: track 167.9 -> 255.2 mm
- net VCC: track 138.3 -> 193.4 mm
- net SDA: track 63.8 -> 45.4 mm
- net N$3: track 10.6 -> 22.0 mm
- net N$2: track 14.3 -> 24.4 mm
- net N$1: track 18.5 -> 28.2 mm
- net N$4: track 7.85 -> 17.3 mm
- net SDO: track 14.3 -> 6.25 mm
- net SCL: track 60.0 -> 67.3 mm
- net CSB: track 37.9 -> 32.5 mm
- net N$10: track 14.4 -> 9.86 mm
- net N$11: track 15.6 -> 11.3 mm
- net N$9: track 13.9 -> 10.5 mm
- net N$14: track 7.58 -> 10.3 mm
- net N$8: track 13.1 -> 15.6 mm
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Other:
- board size 62.2 x 49.2 mm -> 49.7 x 45.7 mm
