File: pcb/main.sch (EAGLE design)
At the start: 19 parts, among them IC1 PCF8574P, U1 BMP280

Commit message: Update pcb files
Parts:
- removed DIS1: TUXGR_16X2_R2, display-lcd:TUXGR_16X2_R2
Connections:
- net GND: no longer DIS1.D0, DIS1.D1, DIS1.D2, DIS1.D3, DIS1.GND, DIS1.NC@2
- net N$1: no longer DIS1.D7
- net N$12: no longer DIS1.CONTR
- net N$14: no longer DIS1.NC@1
- net N$2: no longer DIS1.D6
- net N$3: no longer DIS1.D5
- net N$4: no longer DIS1.D4
- net N$5: no longer DIS1.RS
- net N$7: no longer DIS1.R/W
- net N$8: no longer DIS1.E
- net VCC: no longer DIS1.VCC
Changed lines of the file:
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@@
 <part name="C1" library="rcl" library_urn="urn:adsk.eagle:library:334" deviceset="CPOL-EU" device="E2-5" package3d_urn="urn:adsk.eagle:package:23346/2" value="1uF"/>
 <part name="C2" library="rcl" library_urn="urn:adsk.eagle:library:334" deviceset="CPOL-EU" device="E2-5" package3d_urn="urn:adsk.eagle:package:23346/2" value="0.1uF"/>
-<part name="DIS1" library="display-lcd" library_urn="urn:adsk.eagle:library:214" deviceset="TUXGR_16X2_R2" device="" package3d_urn="urn:adsk.eagle:package:13139/1"/>
 <part name="IC1" library="micro-philips" library_urn="urn:adsk.eagle:library:290" deviceset="PCF8574" device="P" package3d_urn="urn:adsk.eagle:package:20171/1" override_package3d_urn="urn:adsk.eagle:package:30881106/4" override_package_urn="urn:adsk.eagle:footprint:20071/1" value="PCF8574P"/>
 <part name="GND1" library="supply1" library_urn="urn:adsk.eagle:library:371" deviceset="GNDA" device=""/>
@@
 <attribute name="VALUE" x="59.563" y="74.1426" size="1.778" layer="96"/>
 </instance>
-<instance part="DIS1" gate="G$1" x="208.28" y="-66.04" smashed="yes" rot="R180">
-<attribute name="NAME" x="228.6" y="-80.01" size="1.778" layer="95" rot="R180"/>
-<attribute name="VALUE" x="209.55" y="-80.01" size="1.778" layer="96" rot="R180"/>
-</instance>
 <instance part="IC1" gate="G$1" x="170.18" y="-5.08" smashed="yes">
 <attribute name="NAME" x="162.56" y="11.43" size="1.778" layer="95"/>
@@
 <pinref part="R4" gate="G$1" pin="1"/>
 <junction x="-22.86" y="81.28"/>
-<label x="-30.48" y="81.28" size="1.778" layer="95"/>
+<label x="-33.02" y="81.28" size="1.778" layer="95"/>
 </segment>
 <segment>
@@
 </segment>
 <segment>
-<pinref part="DIS1" gate="G$1" pin="D3"/>
-<wire x1="203.2" y1="-55.88" x2="203.2" y2="-50.8" width="0.1524" layer="91"/>
-<pinref part="DIS1" gate="G$1" pin="D0"/>
 <wire x1="203.2" y1="-50.8" x2="205.74" y2="-50.8" width="0.1524" layer="91"/>
 <wire x1="205.74" y1="-50.8" x2="208.28" y2="-50.8" width="0.1524" layer="91"/>
 <wire x1="208.28" y1="-50.8" x2="210.82" y2="-50.8" width="0.1524" layer="91"/>
-<wire x1="210.82" y1="-50.8" x2="210.82" y2="-55.88" width="0.1524" layer="91"/>
-<pinref part="DIS1" gate="G$1" pin="D2"/>
-<wire x1="205.74" y1="-55.88" x2="205.74" y2="-50.8" width="0.1524" layer="91"/>
 <junction x="205.74" y="-50.8"/>
-<pinref part="DIS1" gate="G$1" pin="D1"/>
-<wire x1="208.28" y1="-55.88" x2="208.28" y2="-50.8" width="0.1524" layer="91"/>
 <junction x="208.28" y="-50.8"/>
-<pinref part="DIS1" gate="G$1" pin="GND"/>
 <wire x1="210.82" y1="-50.8" x2="226.06" y2="-50.8" width="0.1524" layer="91"/>
-<wire x1="226.06" y1="-50.8" x2="226.06" y2="-55.88" width="0.1524" layer="91"/>
 <junction x="210.82" y="-50.8"/>
 <wire x1="226.06" y1="-50.8" x2="236.22" y2="-50.8" width="0.1524" layer="91"/>
@@
 <pinref part="R5" gate="G$1" pin="1"/>
 <wire x1="236.22" y1="-48.26" x2="236.22" y2="-50.8" width="0.1524" layer="91"/>
-<pinref part="DIS1" gate="G$1" pin="NC@2"/>
-<wire x1="187.96" y1="-55.88" x2="187.96" y2="-50.8" width="0.1524" layer="91"/>
 <wire x1="187.96" y1="-50.8" x2="203.2" y2="-50.8" width="0.1524" layer="91"/>
 <junction x="203.2" y="-50.8"/>
@@
 <label x="236.22" y="-53.34" size="1.778" layer="95" rot="R180"/>
 <pinref part="JP2" gate="A" pin="1"/>
-<wire x1="226.06" y1="-96.52" x2="226.06" y2="-55.88" width="0.1524" layer="91"/>
-<junction x="226.06" y="-55.88"/>
+<wire x1="226.06" y1="-96.52" x2="226.06" y2="-50.8" width="0.1524" layer="91"/>
 <pinref part="JP2" gate="A" pin="8"/>
-<wire x1="208.28" y1="-96.52" x2="208.28" y2="-55.88" width="0.1524" layer="91"/>
-<junction x="208.28" y="-55.88"/>
+<wire x1="208.28" y1="-96.52" x2="208.28" y2="-50.8" width="0.1524" layer="91"/>
 <pinref part="JP2" gate="A" pin="7"/>
-<wire x1="210.82" y1="-96.52" x2="210.82" y2="-55.88" width="0.1524" layer="91"/>
-<junction x="210.82" y="-55.88"/>
+<wire x1="210.82" y1="-96.52" x2="210.82" y2="-50.8" width="0.1524" layer="91"/>
 <pinref part="JP2" gate="A" pin="9"/>
-<wire x1="205.74" y1="-96.52" x2="205.74" y2="-55.88" width="0.1524" layer="91"/>
-<junction x="205.74" y="-55.88"/>
+<wire x1="205.74" y1="-96.52" x2="205.74" y2="-50.8" width="0.1524" layer="91"/>
 <pinref part="JP2" gate="A" pin="10"/>
-<wire x1="203.2" y1="-96.52" x2="203.2" y2="-55.88" width="0.1524" layer="91"/>
-<junction x="203.2" y="-55.88"/>
+<wire x1="203.2" y1="-96.52" x2="203.2" y2="-50.8" width="0.1524" layer="91"/>
 <pinref part="JP2" gate="A" pin="16"/>
-<wire x1="187.96" y1="-96.52" x2="187.96" y2="-55.88" width="0.1524" layer="91"/>
-<junction x="187.96" y="-55.88"/>
+<wire x1="187.96" y1="-96.52" x2="187.96" y2="-50.8" width="0.1524" layer="91"/>
 </segment>
 <segment>
@@
 </segment>
 <segment>
-<pinref part="DIS1" gate="G$1" pin="VCC"/>
-<wire x1="223.52" y1="-55.88" x2="223.52" y2="-33.02" width="0.1524" layer="91"/>
 <wire x1="223.52" y1="-33.02" x2="236.22" y2="-33.02" width="0.1524" layer="91"/>
 <pinref part="R5" gate="G$1" pin="2"/>
@@
 <label x="238.76" y="-35.56" size="1.778" layer="95"/>
 <pinref part="JP2" gate="A" pin="2"/>
-<wire x1="223.52" y1="-96.52" x2="223.52" y2="-55.88" width="0.1524" layer="91"/>
-<junction x="223.52" y="-55.88"/>
+<wire x1="223.52" y1="-96.52" x2="223.52" y2="-33.02" width="0.1524" layer="91"/>
 </segment>
 <segment>
@@
 <segment>
 <pinref part="IC1" gate="G$1" pin="P7"/>
-<pinref part="DIS1" gate="G$1" pin="D7"/>
 <wire x1="182.88" y1="-15.24" x2="193.04" y2="-15.24" width="0.1524" layer="91"/>
-<wire x1="193.04" y1="-15.24" x2="193.04" y2="-55.88" width="0.1524" layer="91"/>
 <pinref part="JP2" gate="A" pin="14"/>
-<wire x1="193.04" y1="-96.52" x2="193.04" y2="-55.88" width="0.1524" layer="91"/>
-<junction x="193.04" y="-55.88"/>
+<wire x1="193.04" y1="-96.52" x2="193.04" y2="-15.24" width="0.1524" layer="91"/>
 </segment>
 </net>
@@
 <segment>
 <pinref part="IC1" gate="G$1" pin="P6"/>
-<pinref part="DIS1" gate="G$1" pin="D6"/>
 <wire x1="182.88" y1="-12.7" x2="195.58" y2="-12.7" width="0.1524" layer="91"/>
-<wire x1="195.58" y1="-12.7" x2="195.58" y2="-55.88" width="0.1524" layer="91"/>
+<wire x1="195.58" y1="-12.7" x2="195.58" y2="-96.52" width="0.1524" layer="91"/>
 <pinref part="JP2" gate="A" pin="13"/>
-<wire x1="195.58" y1="-96.52" x2="195.58" y2="-55.88" width="0.1524" layer="91"/>
-<junction x="195.58" y="-55.88"/>
 </segment>
 </net>
@@
 <segment>
 <pinref part="IC1" gate="G$1" pin="P5"/>
-<pinref part="DIS1" gate="G$1" pin="D5"/>
 <wire x1="182.88" y1="-10.16" x2="198.12" y2="-10.16" width="0.1524" layer="91"/>
-<wire x1="198.12" y1="-10.16" x2="198.12" y2="-55.88" width="0.1524" layer="91"/>
+<wire x1="198.12" y1="-10.16" x2="198.12" y2="-96.52" width="0.1524" layer="91"/>
 <pinref part="JP2" gate="A" pin="12"/>
-<wire x1="198.12" y1="-96.52" x2="198.12" y2="-55.88" width="0.1524" layer="91"/>
-<junction x="198.12" y="-55.88"/>
 </segment>
 </net>
@@
 <segment>
 <pinref part="IC1" gate="G$1" pin="P4"/>
-<pinref part="DIS1" gate="G$1" pin="D4"/>
 <wire x1="182.88" y1="-7.62" x2="200.66" y2="-7.62" width="0.1524" layer="91"/>
-<wire x1="200.66" y1="-7.62" x2="200.66" y2="-55.88" width="0.1524" layer="91"/>
+<wire x1="200.66" y1="-7.62" x2="200.66" y2="-96.52" width="0.1524" layer="91"/>
 <pinref part="JP2" gate="A" pin="11"/>
-<wire x1="200.66" y1="-96.52" x2="200.66" y2="-55.88" width="0.1524" layer="91"/>
-<junction x="200.66" y="-55.88"/>
 </segment>
 </net>
 <net name="N$5" class="0">
 <segment>
-<pinref part="DIS1" gate="G$1" pin="RS"/>
 <pinref part="IC1" gate="G$1" pin="P0"/>
-<wire x1="218.44" y1="-55.88" x2="218.44" y2="2.54" width="0.1524" layer="91"/>
+<wire x1="218.44" y1="-96.52" x2="218.44" y2="2.54" width="0.1524" layer="91"/>
 <wire x1="218.44" y1="2.54" x2="182.88" y2="2.54" width="0.1524" layer="91"/>
 <pinref part="JP2" gate="A" pin="4"/>
-<wire x1="218.44" y1="-96.52" x2="218.44" y2="-55.88" width="0.1524" layer="91"/>
-<junction x="218.44" y="-55.88"/>
 </segment>
 </net>
 <net name="N$7" class="0">
 <segment>
-<pinref part="DIS1" gate="G$1" pin="R/W"/>
 <pinref part="IC1" gate="G$1" pin="P1"/>
-<wire x1="215.9" y1="-55.88" x2="215.9" y2="0" width="0.1524" layer="91"/>
+<wire x1="215.9" y1="-96.52" x2="215.9" y2="0" width="0.1524" layer="91"/>
 <wire x1="215.9" y1="0" x2="182.88" y2="0" width="0.1524" layer="91"/>
 <pinref part="JP2" gate="A" pin="5"/>
-<wire x1="215.9" y1="-96.52" x2="215.9" y2="-55.88" width="0.1524" layer="91"/>
-<junction x="215.9" y="-55.88"/>
 </segment>
 </net>
 <net name="N$8" class="0">
 <segment>
-<pinref part="DIS1" gate="G$1" pin="E"/>
 <pinref part="IC1" gate="G$1" pin="P2"/>
-<wire x1="213.36" y1="-55.88" x2="213.36" y2="-2.54" width="0.1524" layer="91"/>
+<wire x1="213.36" y1="-96.52" x2="213.36" y2="-2.54" width="0.1524" layer="91"/>
 <wire x1="213.36" y1="-2.54" x2="182.88" y2="-2.54" width="0.1524" layer="91"/>
 <pinref part="JP2" gate="A" pin="6"/>
-<wire x1="213.36" y1="-96.52" x2="213.36" y2="-55.88" width="0.1524" layer="91"/>
-<junction x="213.36" y="-55.88"/>
 </segment>
 </net>
@@
 <segment>
 <pinref part="R11" gate="G$1" pin="2"/>
-<pinref part="DIS1" gate="G$1" pin="NC@1"/>
-<wire x1="190.5" y1="-48.26" x2="190.5" y2="-55.88" width="0.1524" layer="91"/>
 <pinref part="JP2" gate="A" pin="15"/>
-<wire x1="190.5" y1="-96.52" x2="190.5" y2="-55.88" width="0.1524" layer="91"/>
-<junction x="190.5" y="-55.88"/>
+<wire x1="190.5" y1="-96.52" x2="190.5" y2="-48.26" width="0.1524" layer="91"/>
 </segment>
 </net>
@@
 <segment>
 <pinref part="JP2" gate="A" pin="3"/>
-<pinref part="DIS1" gate="G$1" pin="CONTR"/>
 <wire x1="220.98" y1="-96.52" x2="220.98" y2="-55.88" width="0.1524" layer="91"/>
 </segment>
